File: hardware/flight-controller/show-fc.kicad_sch (KiCad schematic)
At the start: 126 parts, among them J1 USB-C, J2 microSD, J3 ESC, J4 GPS, J5 LIGHT, J6 RC, J7 TELEM2, J8 SWD, Q1 2N7002, SW1 BOOT, SW2 RESET, U1 RP2354B, U2 USBLC6-2SC6, U3 LMR51635YDDCR, U4 LP5912-3.3DRVR, U5 LP5912-1.8DRVR, U6 ICM-42688-P, U7 BMI270, U8 DPS368, Y1 12MHz

Commit message: Show FC: routing pipeline, 54 mm board, PCBWay rules and README (routing in progress)
Adds the Freerouting pipeline (route.py), fab export (make_fab.py), the
PCBWay .kicad_dru and the README. Widens the flats to 54 mm (corners
still 27 mm), remaps LED data to GPIO42, moves the AUX and TELEM2 pads
next to their pins and drops SD card detect.

Co-Authored-By: Claude Opus 5.5 (1M context) <noreply@anthropic.com>
Claude-Session: https://claude.ai/code/session_01BR3A1ZEFbsPLQy3Mn5HNY3
Parts:
- removed C35, C36: 100n, Capacitor_SMD:C_0603_1608Metric, symbol showfc:C
- removed J7: TELEM2, Connector_JST:JST_GH_SM04B-GHS-TB_1x04-1MP_P1.25mm_Horizontal, symbol showfc:Conn_01x04_MP
- removed R19, R20, R28, R29, R30: 10k, Resistor_SMD:R_0603_1608Metric, symbol showfc:R
- removed R21: 1k, Resistor_SMD:R_0603_1608Metric, symbol showfc:R
- removed TP14: GND, TestPoint:TestPoint_Pad_D1.5mm, symbol showfc:TP
- C1, C10, C11, C15, C16, C17, C2, C3, C37, C38, C39, C4, C40, C41, C42, C5, C6, C7, C8, C9: footprint Capacitor_SMD:C_0603_1608Metric -> Capacitor_SMD:C_0402_1005Metric; MPN GCM188R71H104KA57D -> GRM155R71C104KA88D
- C19, C20: footprint Capacitor_SMD:C_0603_1608Metric -> Capacitor_SMD:C_0402_1005Metric; MPN GRM1885C1H150JA01D -> GRM1555C1H150JA01D
- D3: value SMAJ30A -> SMF30A; footprint Diode_SMD:D_SMA -> Diode_SMD:D_SOD-123F; MPN SMAJ30A -> SMF30A
- R10, R9: footprint Resistor_SMD:R_0603_1608Metric -> Resistor_SMD:R_0402_1005Metric; MPN RC0603FR-0727L -> RC0402FR-0727L
- R2: footprint Resistor_SMD:R_0603_1608Metric -> Resistor_SMD:R_0402_1005Metric; MPN RC0603FR-071KL -> RC0402FR-071KL
- R22, R23: footprint Resistor_SMD:R_0603_1608Metric -> Resistor_SMD:R_0402_1005Metric; MPN RC0603FR-0710KL -> RC0402FR-0710KL
- R24, R25: footprint Resistor_SMD:R_0603_1608Metric -> Resistor_SMD:R_0402_1005Metric; MPN RC0603FR-072R2KL -> RC0402FR-072R2KL
- TP1, TP2: footprint TestPoint:TestPoint_Pad_D2.0mm -> TestPoint:TestPoint_Pad_D1.5mm
- TP10: value ADC_SPARE_IN -> +3V3
- TP11: value GPIO44 -> GND
- TP12: value GPIO45 -> TEL2_TX
- TP13: value +3V3 -> TEL2_RX
- U4, U5: footprint Package_SON:WSON-6-1EP_2x2mm_P0.65mm_EP1x1.6mm -> Package_SON:WSON-6-1EP_2x2mm_P0.65mm_EP1x1.6mm_ThermalVias
Connections:
- net ADC_5V is gone; now on net LED_DATA: U1.53 (GPIO42/ADC2)
- net ADC_SPARE_IN is gone; now on net +3V3: TP10.1
- net +3V3: no longer TP13.1
- net GND: now also TP11.1
- net LED_DATA: no longer U1.28 (GPIO27)
- net TEL2_RX: now also TP13.1
- net TEL2_TX: now also TP12.1
- net ADC_SPARE: no longer names the net of U1.54 (GPIO43/ADC3)
- net GPIO44: no longer names the net of U1.55 (GPIO44/ADC4)
- net GPIO44: no longer TP11.1
- net GPIO45: no longer names the net of U1.56 (GPIO45/ADC5)
- net GPIO45: no longer TP12.1
- net SD_DAT1: no longer names the net of J2.8 (DAT1)
- net SD_DAT2: no longer names the net of J2.1 (DAT2)
- net SD_DET: no longer names the net of J2.9 (DET_B)
- net SD_DET: no longer U1.46 (GPIO37)
- no-connect marks 18 -> 26
Other:
- moved on the sheet: C43, C44, D7, Q1, R31, R32, R33, R34, R35, TP1, TP10, TP11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

Commit message: Show FC: routed 54 mm board (4 connections left), stacking holes, fab outputs
Routes the 2-layer board with Freerouting plus a second pass (finish.py);
four connections remain for KiCad's interactive router, listed in the
README. Mounting holes follow the shared stack spec (3.3 mm unplated,
30.5 mm pattern, 7.5 mm copper-free ring). Adds Gerbers, drill, CPL and
BOM in fab/ and board renders.

Co-Authored-By: Claude Opus 5.5 (1M context) <noreply@anthropic.com>
Claude-Session: https://claude.ai/code/session_01BR3A1ZEFbsPLQy3Mn5HNY3
Parts:
- H1, H2, H3, H4: footprint MountingHole:MountingHole_3.2mm_M3 -> showfc:MountingHole_3.3mm_M3_Stack
Changed lines of the file:
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@@
       (effects (font (size 1.27 1.27)) (justify left))
     )
-    (property "Footprint" "MountingHole:MountingHole_3.2mm_M3" (at 670.56 424.18 0)
+    (property "Footprint" "showfc:MountingHole_3.3mm_M3_Stack" (at 670.56 424.18 0)
       (effects (font (size 1.27 1.27)) (justify left) hide)
     )
@@
       (effects (font (size 1.27 1.27)) (justify left))
     )
-    (property "Footprint" "MountingHole:MountingHole_3.2mm_M3" (at 688.34 424.18 0)
+    (property "Footprint" "showfc:MountingHole_3.3mm_M3_Stack" (at 688.34 424.18 0)
       (effects (font (size 1.27 1.27)) (justify left) hide)
     )
@@
       (effects (font (size 1.27 1.27)) (justify left))
     )
-    (property "Footprint" "MountingHole:MountingHole_3.2mm_M3" (at 706.12 424.18 0)
+    (property "Footprint" "showfc:MountingHole_3.3mm_M3_Stack" (at 706.12 424.18 0)
       (effects (font (size 1.27 1.27)) (justify left) hide)
     )
@@
       (effects (font (size 1.27 1.27)) (justify left))
     )
-    (property "Footprint" "MountingHole:MountingHole_3.2mm_M3" (at 723.9 424.18 0)
+    (property "Footprint" "showfc:MountingHole_3.3mm_M3_Stack" (at 723.9 424.18 0)
       (effects (font (size 1.27 1.27)) (justify left) hide)
     )

Commit message: Show FC: finish routing, add SWD debug pads, move project to KiCad 10
- Upgrade schematic, board and project to the KiCad 10 format. The schematic
  now uses global labels so its net names match the board's, and the TP
  symbol pin sits on the 1.27 mm grid; ERC is clean.
- Route the last four connections by hand:
  XOUT from U1.31 between XIN and +1V1, under Y1 to R2 (XIN narrowed to 0.15);
  USB_DP from R9 through a via inside the U2 loop, bottom layer to a via over
  U1.67 (USB_DM via and the +1V1 core link moved to make room);
  VBAT by swapping R16 and R17, so R16's VBAT pad sits beside C24;
  BUZZER from U1.27 around the mounting holes on the bottom layer to R34.
- Add five 1 mm SWD debug pads (TP14-TP18: SWDIO, GND, SWCLK, 3V3, RUN) on
  the bottom behind J8, in design.py and the schematic as test points.
- Remove two dangling stubs, set solid zone connections on four starved
  thermals. DRC with parity and zone refill: 0 errors, 0 warnings,
  0 unconnected.
- Regenerate fab outputs and renders with KiCad 10; update the README.
- handroute.py: GRID, SLACK and SIGNAL_W can be set from the environment.

Co-Authored-By: Claude Opus 5.5 (1M context) <noreply@anthropic.com>
Claude-Session: https://claude.ai/code/session_01BR3A1ZEFbsPLQy3Mn5HNY3
Parts:
- added TP14: SWDIO, TestPoint:TestPoint_Pad_D1.0mm, symbol showfc:TP
- added TP15: GND, TestPoint:TestPoint_Pad_D1.0mm, symbol showfc:TP
- added TP16: SWCLK, TestPoint:TestPoint_Pad_D1.0mm, symbol showfc:TP
- added TP17: +3V3, TestPoint:TestPoint_Pad_D1.0mm, symbol showfc:TP
- added TP18: RUN, TestPoint:TestPoint_Pad_D1.0mm, symbol showfc:TP
Connections:
- net +3V3: now also TP17.1
- net GND: now also TP15.1
- net RUN: now also TP18.1
- net SWCLK: now also TP16.1
- net SWDIO: now also TP14.1
