File: hardware/esc/ESC.kicad_sch (KiCad schematic)
At the start: 36 parts, among them Q1 SP40N01GHNK, Q11 SP40N01GHNK, Q16 SP40N01GHNK, Q2 SP40N01GHNK, Q21 SP40N01GHNK, Q6 SP40N01GHNK, U2 AT32F421G8U7, U4 NSG2065Q

Commit message: esc: 0402 passives round each MCU, side-entry JST SH for the FC lead
The decoupling, NRST, BOOT0, VDDA, back-EMF divider and DShot parts round
each AT32F421 go from 0603 to 0402 (YAGEO RC0402, Samsung CL05B104KB5NNNC),
so the MCU can move inboard next to its gate driver with room for its
escape tracks. Gate resistors, bootstrap and driver supply caps stay 0603.

J1 becomes the side-entry SM08B-SRSS-TB (LCSC C160407; the old C160390 was a
4-pin BM04B), so the FC lead leaves the board edge sideways instead of
standing up into the stack.

tools/schematic_0402.py is the one-shot script that made the change.

Co-Authored-By: Claude Opus 5.5 (1M context) <noreply@anthropic.com>
Claude-Session: https://claude.ai/code/session_015X7Az2AeDtDrTq19qE6e7H
Parts:
- C48, C49, C50: footprint Capacitor_SMD:C_0603_1608Metric -> Capacitor_SMD:C_0402_1005Metric; MPN CL10B104KB8NNNC -> CL05B104KB5NNNC
- R18, R19, R25, R27, R28, R30, R31, R33: footprint Resistor_SMD:R_0603_1608Metric -> Resistor_SMD:R_0402_1005Metric; MPN RC0603FR-0710KL -> RC0402FR-0710KL
- R20: footprint Resistor_SMD:R_0603_1608Metric -> Resistor_SMD:R_0402_1005Metric; MPN RC0603FR-07220RL -> RC0402FR-07220RL
- R26, R29, R32: footprint Resistor_SMD:R_0603_1608Metric -> Resistor_SMD:R_0402_1005Metric; MPN RC0603FR-071KL -> RC0402FR-071KL
- R84: footprint Resistor_SMD:R_0603_1608Metric -> Resistor_SMD:R_0402_1005Metric; MPN RC0603FR-0710RL -> RC0402FR-0710RL
