File: hardware/esc/drone-esc.kicad_sch (KiCad schematic)
At the start: 53 parts, among them J1 BM08B-SRSS-TB, U12 INA186A3IDCKR, U13 LMR54406DBVR, U14 FTC160808S4R7MBCA, U15 TLV76733DRVR

Commit message: esc: 0402 passives round each MCU, side-entry JST SH for the FC lead
The decoupling, NRST, BOOT0, VDDA, back-EMF divider and DShot parts round
each AT32F421 go from 0603 to 0402 (YAGEO RC0402, Samsung CL05B104KB5NNNC),
so the MCU can move inboard next to its gate driver with room for its
escape tracks. Gate resistors, bootstrap and driver supply caps stay 0603.

J1 becomes the side-entry SM08B-SRSS-TB (LCSC C160407; the old C160390 was a
4-pin BM04B), so the FC lead leaves the board edge sideways instead of
standing up into the stack.

tools/schematic_0402.py is the one-shot script that made the change.

Co-Authored-By: Claude Opus 5.5 (1M context) <noreply@anthropic.com>
Claude-Session: https://claude.ai/code/session_015X7Az2AeDtDrTq19qE6e7H
Parts:
- J1: value BM08B-SRSS-TB -> SM08B-SRSS-TB; footprint drone-esc:JST_SH_BM08B-SRSS-TB_Vertical -> drone-esc:JST_SH_SM08B-SRSS-TB_Horizontal; LCSC C160390 -> C160407; MPN BM08B-SRSS-TB(LF)(SN) -> SM08B-SRSS-TB(LF)(SN)
